File: hardware_test.kicad_sch (KiCad schematic)
At the start: 1 part, among them U1 4002

Commit message: Test modify
Parts:
- removed U1: 4002, symbol 4xxx:4002
Changed lines of the file:
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@@
 	(generator_version "9.0")
 	(paper "A4")
-	(symbol
-		(lib_id "4xxx:4002")
-		(at 81.28 66.04 0)
-		(unit 1)
-		(exclude_from_sim no)
-		(in_bom yes)
-		(on_board yes)
-		(dnp no)
-		(fields_autoplaced yes)
-		(property "Reference" "U1"
-			(at 81.28 57.15 0)
-			(effects
-				(font
-					(size 1.27 1.27)
-				)
-			)
-		)
-		(property "Value" "4002"
-			(at 81.28 59.69 0)
-			(effects
-				(font
-					(size 1.27 1.27)
-				)
-			)
-		)
-		(property "Footprint" ""
-			(at 81.28 66.04 0)
-			(effects
-				(font
-					(size 1.27 1.27)
-				)
-				(hide yes)
-			)
-		)
-		(property "Datasheet" "http://www.intersil.com/content/dam/Intersil/documents/cd40/cd4000bms-01bms-02bms-25bms.pdf"
-			(at 81.28 66.04 0)
-			(effects
-				(font
-					(size 1.27 1.27)
-				)
-				(hide yes)
-			)
-		)
-		(property "Description" "Dual  4 input NOR gate"
-			(at 81.28 66.04 0)
-			(effects
-				(font
-					(size 1.27 1.27)
-				)
-				(hide yes)
-			)
-		)
-		(pin "14"
-		)
-		(pin "10"
-		)
-		(pin "9"
-		)
-		(pin "1"
-		)
-		(pin "5"
-		)
-		(pin "3"
-		)
-		(pin "2"
-		)
-		(pin "4"
-		)
-		(pin "13"
-		)
-		(pin "12"
-		)
-		(pin "7"
-		)
-		(pin "11"
-		)
-		(instances
-			(project ""
-				(path "/410f0359-07d5-42e8-b1f6-46111181664c"
-					(reference "U1")
-					(unit 1)
-				)
-			)
-		)
-	)
 	(sheet_instances
 		(path "/"
